Commit message: ur10 with tool

File: data/robot_description/ur5_with_measurement_tool/urdf/ur5_with_measurement_tool.urdf (robot description, URDF)
Before this commit: robot ur5_with_measurement_tool, 13 links, 12 joints
Links:
- link base_link: geometry collision mesh filename=package://ur_description/meshes/ur5/collision/base.stl; visual mesh filename=package://ur_description/meshes/ur5/visual/base.obj
- link forearm_link: geometry collision mesh filename=package://ur_description/meshes/ur5/collision/forearm.stl; visual mesh filename=package://ur_description/meshes/ur5/visual/forearm.obj
- link shoulder_link: geometry collision mesh filename=package://ur_description/meshes/ur5/collision/shoulder.stl; visual mesh filename=package://ur_description/meshes/ur5/visual/shoulder.obj
- link upper_arm_link: geometry collision mesh filename=package://ur_description/meshes/ur5/collision/upperarm.stl; visual mesh filename=package://ur_description/meshes/ur5/visual/upperarm.obj
- link wrist_1_link: geometry collision mesh filename=package://ur_description/meshes/ur5/collision/wrist1.stl; visual mesh filename=package://ur_description/meshes/ur5/visual/wrist1.obj
- link wrist_2_link: geometry collision mesh filename=package://ur_description/meshes/ur5/collision/wrist2.stl; visual mesh filename=package://ur_description/meshes/ur5/visual/wrist2.obj
- link wrist_3_link: geometry collision mesh filename=package://ur_description/meshes/ur5/collision/wrist3.stl; visual mesh filename=package://ur_description/meshes/ur5/visual/wrist3.obj

File: data/robot_description/ur_description/urdf/ur10.urdf (robot description, URDF)
Before this commit: robot ur10, 11 links, 10 joints
Links:
- link base_link: geometry collision mesh filename=package://ur_description/meshes/ur10/collision/base.stl; visual mesh filename=package://ur_description/meshes/ur10/visual/_base.obj
- link forearm_link: geometry collision mesh filename=package://ur_description/meshes/ur10/collision/forearm.stl; visual mesh filename=package://ur_description/meshes/ur10/visual/_forearm.obj
- link shoulder_link: geometry collision mesh filename=package://ur_description/meshes/ur10/collision/shoulder.stl; visual mesh filename=package://ur_description/meshes/ur10/visual/_shoulder.obj
- link upper_arm_link: geometry collision mesh filename=package://ur_description/meshes/ur10/collision/upperarm.stl; visual mesh filename=package://ur_description/meshes/ur10/visual/_upperarm.obj
- link wrist_1_link: geometry collision mesh filename=package://ur_description/meshes/ur10/collision/wrist1.stl; visual mesh filename=package://ur_description/meshes/ur10/visual/_wrist1.obj
- link wrist_2_link: geometry collision mesh filename=package://ur_description/meshes/ur10/collision/wrist2.stl; visual mesh filename=package://ur_description/meshes/ur10/visual/_wrist2.obj
- link wrist_3_link: geometry collision mesh filename=package://ur_description/meshes/ur10/collision/wrist3.stl; visual mesh filename=package://ur_description/meshes/ur10/visual/_wrist3.obj
