Commit message: fixed ur3_rot and added to example files

File: data/robot_description/ur_description/urdf/ur3_rot.urdf (robot description, URDF)
Before this commit: robot ur3, 11 links, 10 joints
Joints:
- joint ee_fixed_joint: origin xyz=0.0 0.0819 0.0 rpy=0.0 0.0 1.57079632679 -> xyz=0.0 0.0819 0.0 rpy=-1.57079632679 0.0 0.0
- joint shoulder_pan_joint: axis 0 1 0 -> 0 0 1; origin xyz=0.0 0.0 0.1519 rpy=0.0 0.0 0.0 -> xyz=0.0 0.0 0.1519 rpy=0.0 0.0 -3.14159265359
